File: IREC-FlighComputer.kicad_pcb (KiCad board)
At the start: 4 copper layers, 109 x 59 mm, 148 parts, among them IC1 SN74HCT125DR, J1 Molex Microfit, J10 Conn_01x03_Socket, J2 Conn_01x03_Socket, J3 RF2-04A-T-00-50-G, J4 Conn_02x04_Counter_Clockwise, J5 BMI-S-209-F, J7 Conn_01x02_Socket, J8 Conn_01x02_Socket, Q4 SI7232DN-T1-GE3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

Commit message: add silk screen
Parts:
- added LOGO: LOGO, LOGO, B.Cu at (150.2, 89.8)
Other:
- board text added: "Taspol S. CURSR-IV Flight Computer"
